Commit message: collision 연습할 파일 복사

File: src/QUB_urdf/urdf/QUB v1.2 collision.urdf (robot description, URDF)
Before this commit: robot QUB v1.2_urdf_4th, 14 links, 13 joints
Links:
- link L_ankle_link: geometry collision mesh filename=file:///Users/jae/Library/Mobile Documents/com~apple~CloudD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; visual mesh filename=file:///Users/jae/Library/Mobile Documents/com~apple~CloudD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
- link L_calf_link: geometry collision mesh filename=file:///Users/jae/Library/Mobile Documents/com~apple~CloudD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; visual mesh filename=file:///Users/jae/Library/Mobile Documents/com~apple~CloudD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
- link L_foot_link: geometry collision mesh filename=file:///Users/jae/Library/Mobile Documents/com~apple~CloudD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; visual mesh filename=file:///Users/jae/Library/Mobile Documents/com~apple~CloudD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
- link L_hip_r_link: geometry collision mesh filename=file:///Users/jae/Library/Mobile Documents/com~apple~CloudD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; visual mesh filename=file:///Users/jae/Library/Mobile Documents/com~apple~CloudD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
- link L_hip_y_link: geometry collision mesh filename=file:///Users/jae/Library/Mobile Documents/com~apple~CloudD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; visual mesh filename=file:///Users/jae/Library/Mobile Documents/com~apple~CloudD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
- link L_thigh_link: geometry collision mesh filename=file:///Users/jae/Library/Mobile Documents/com~apple~CloudD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; visual mesh filename=file:///Users/jae/Library/Mobile Documents/com~apple~CloudD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
- link R_ankle_link: geometry collision mesh filename=file:///Users/jae/Library/Mobile Documents/com~apple~CloudD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; visual mesh filename=file:///Users/jae/Library/Mobile Documents/com~apple~CloudD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
- link R_calf_link: geometry collision mesh filename=file:///Users/jae/Library/Mobile Documents/com~apple~CloudD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; visual mesh filename=file:///Users/jae/Library/Mobile Documents/com~apple~CloudD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
- link R_foot_link: geometry collision mesh filename=file:///Users/jae/Library/Mobile Documents/com~apple~CloudD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; visual mesh filename=file:///Users/jae/Library/Mobile Documents/com~apple~CloudD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
- link R_hip_r_link: geometry collision mesh filename=file:///Users/jae/Library/Mobile Documents/com~apple~CloudD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; visual mesh filename=file:///Users/jae/Library/Mobile Documents/com~apple~CloudD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
- link R_hip_y_link: geometry collision mesh filename=file:///Users/jae/Library/Mobile Documents/com~apple~CloudD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; visual mesh filename=file:///Users/jae/Library/Mobile Documents/com~apple~CloudD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
- link R_thigh_link: geometry collision mesh filename=file:///Users/jae/Library/Mobile Documents/com~apple~CloudD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; visual mesh filename=file:///Users/jae/Library/Mobile Documents/com~apple~CloudD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
- link base_link: geometry collision mesh filename=file:///Users/jae/Library/Mobile Documents/com~apple~CloudD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; visual mesh filename=file:///Users/jae/Library/Mobile Documents/com~apple~CloudD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
- link pelvis_link: geometry collision mesh filename=file:///Users/jae/Library/Mobile Documents/com~apple~CloudD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; visual mesh filename=file:///Users/jae/Library/Mobile Documents/com~apple~CloudD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
