Commit message: 물성치 적용 완료

File: src/QUB_urdf/urdf/QUB v1.2_@Mac.urdf (robot description, URDF)
Before this commit: robot QUB, 14 links, 13 joints
Links:
- link L_ankle_link: mass 0.0236524344915325 -> 0.02200
- link L_calf_link: mass 1.17074765561419 -> 1.97157
- link L_foot_link: mass 0.359946537295079 -> 0.25200
- link L_hip_r_link: mass 0.855798957044734 -> 1.24854
- link L_hip_y_link: mass 0.917755275631564 -> 1.32879
- link L_thigh_link: mass 1.37472432263504 -> 2.18164
- link R_ankle_link: mass 0.0236524344915325 -> 0.02200
- link R_calf_link: mass 1.17074722849011 -> 1.97157
- link R_foot_link: mass 0.359946538045687 -> 0.25200
- link R_hip_r_link: mass 0.855799021923541 -> 1.24854
- link R_hip_y_link: mass 0.9177638118792 -> 1.32879
- link R_thigh_link: mass 1.3747257194995 -> 2.18164
- link base_link: mass 4.07254209371122 -> 4.21449
- link pelvis_link: mass 2.18597276276807 -> 3.69660
