Commit message: GPU용 파일 수정

File: src/QUB_urdf/urdf/QUB v1.2_@GPU.urdf (robot description, URDF)
Before this commit: robot QUB, 14 links, 13 joints
Links:
- link L_ankle_link: geometry collision mesh filename=file:///home/qub1/Jaebin/URDF_study/src/QUB_urdf/meshes/col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; visual mesh filename=file:///home/qub1/Jaebin/URDF_study/src/QUB_urdf/meshes/L_a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
- link L_calf_link: geometry collision mesh filename=file:///home/qub1/Jaebin/URDF_study/src/QUB_urdf/meshes/col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; visual mesh filename=file:///home/qub1/Jaebin/URDF_study/src/QUB_urdf/meshes/L_c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
- link L_foot_link: geometry collision mesh filename=file:///home/qub1/Jaebin/URDF_study/src/QUB_urdf/meshes/col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; visual mesh filename=file:///home/qub1/Jaebin/URDF_study/src/QUB_urdf/meshes/L_f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
- link L_hip_r_link: geometry collision mesh filename=file:///home/qub1/Jaebin/URDF_study/src/QUB_urdf/meshes/col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; visual mesh filename=file:///home/qub1/Jaebin/URDF_study/src/QUB_urdf/meshes/L_h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
- link L_hip_y_link: geometry collision mesh filename=file:///home/qub1/Jaebin/URDF_study/src/QUB_urdf/meshes/col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; visual mesh filename=file:///home/qub1/Jaebin/URDF_study/src/QUB_urdf/meshes/L_h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
- link L_thigh_link: geometry collision mesh filename=file:///home/qub1/Jaebin/URDF_study/src/QUB_urdf/meshes/col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; visual mesh filename=file:///home/qub1/Jaebin/URDF_study/src/QUB_urdf/meshes/L_t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
- link R_ankle_link: geometry collision mesh filename=file:///home/qub1/Jaebin/URDF_study/src/QUB_urdf/meshes/col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; visual mesh filename=file:///home/qub1/Jaebin/URDF_study/src/QUB_urdf/meshes/R_a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
- link R_calf_link: geometry collision mesh filename=file:///home/qub1/Jaebin/URDF_study/src/QUB_urdf/meshes/col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; visual mesh filename=file:///home/qub1/Jaebin/URDF_study/src/QUB_urdf/meshes/R_c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
- link R_foot_link: geometry collision mesh filename=file:///home/qub1/Jaebin/URDF_study/src/QUB_urdf/meshes/col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; visual mesh filename=file:///home/qub1/Jaebin/URDF_study/src/QUB_urdf/meshes/R_f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
- link R_hip_r_link: geometry collision mesh filename=file:///home/qub1/Jaebin/URDF_study/src/QUB_urdf/meshes/col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; visual mesh filename=file:///home/qub1/Jaebin/URDF_study/src/QUB_urdf/meshes/R_h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
- link R_hip_y_link: geometry collision mesh filename=file:///home/qub1/Jaebin/URDF_study/src/QUB_urdf/meshes/col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; visual mesh filename=file:///home/qub1/Jaebin/URDF_study/src/QUB_urdf/meshes/R_h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
- link R_thigh_link: geometry collision mesh filename=file:///home/qub1/Jaebin/URDF_study/src/QUB_urdf/meshes/col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; visual mesh filename=file:///home/qub1/Jaebin/URDF_study/src/QUB_urdf/meshes/R_t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
- link base_link: geometry collision box size=0.140 0.200 0.279; visual mesh filename=file:///home/qub1/Jaebin/URDF_study/src/QUB_urdf/meshes/bas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
- link pelvis_link: geometry collision mesh filename=file:///home/qub1/Jaebin/URDF_study/src/QUB_urdf/meshes/col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; visual mesh filename=file:///home/qub1/Jaebin/URDF_study/src/QUB_urdf/meshes/pel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
