Commit message: torso 물리량 수정

File: src/QUB_URDF_fin/urdf/QUB_v1.2_@Mac.urdf (robot description, URDF)
Before this commit: robot QUB v1.2 urdf, 14 links, 13 joints
Links:
- link base_link: mass 4.0725 -> 4.21449

Commit message: pelvis 물성치 수정

File: src/QUB_URDF_fin/urdf/QUB_v1.2_@Mac.urdf (robot description, URDF)
Before this commit: robot QUB v1.2 urdf, 14 links, 13 joints
Links:
- link pelvis_link: mass 2.18597276276807 -> 3.69660

Commit message: hip roll L,R 물성치 수정

File: src/QUB_URDF_fin/urdf/QUB_v1.2_@Mac.urdf (robot description, URDF)
Before this commit: robot QUB v1.2 urdf, 14 links, 13 joints
Links:
- link L_hip_r_link: mass 0.8558 -> 1.24854
- link R_hip_r_link: mass 0.8558 -> 1.24854

Commit message: ankle 물성치 적용

File: src/QUB_URDF_fin/urdf/QUB_v1.2_@Mac.urdf (robot description, URDF)
Before this commit: robot QUB v1.2 urdf, 14 links, 13 joints
Links:
- link L_ankle_link: mass 0.0236524344915326 -> 0.02200
- link R_ankle_link: mass 0.0236524344915325 -> 0.02200

Commit message: foot 물성치 적용

File: src/QUB_URDF_fin/urdf/QUB_v1.2_@Mac.urdf (robot description, URDF)
Before this commit: robot QUB v1.2 urdf, 14 links, 13 joints
Links:
- link L_foot_link: mass 0.359946548540282 -> 0.25200
- link R_foot_link: mass 0.359946548475121 -> 0.25200
